File: schematics/PC.kicad_sch (KiCad schematic)
At the start: 3 parts, among them U28 74LS161, U29 74LS161, U30 74LS161

Commit message: schematics
Parts:
- added D2 (x11): LED, symbol Device:LED
- added R2 (x11): 1k, symbol Device:R
- added U23 (x2): 74LS245, symbol 74xx:74LS245
- added U33: 74LS04, symbol 74xx:74LS04
Connections:
- net MBUS_0: now also U28.3 (D0), D2.2 (A), U23.2 (A0)
- net MBUS_1: now also U28.4 (D1), D2.2 (A), U23.3 (A1)
- net MBUS_10: now also U30.5 (D2), D2.2 (A), U23.4 (A2)
- net MBUS_2: now also U28.5 (D2), D2.2 (A), U23.4 (A2)
- net MBUS_3: now also U28.6 (D3), D2.2 (A), U23.5 (A3)
- net MBUS_4: now also U29.3 (D0), D2.2 (A), U23.6 (A4)
- net MBUS_5: now also U29.4 (D1), D2.2 (A), U23.7 (A5)
- net MBUS_6: now also U29.5 (D2), D2.2 (A), U23.8 (A6)
- net MBUS_7: now also U29.6 (D3), D2.2 (A), U23.9 (A7)
- net MBUS_8: now also U30.3 (D0), D2.2 (A), U23.2 (A0)
- net MBUS_9: now also U30.4 (D1), D2.2 (A), U23.3 (A1)
- net PC_RST: now reaches U29.1 (~{MR})
- net PC_RST: now also U28.1 (~{MR}), U30.1 (~{MR}), U33.2
- net PC_EN: now reaches U29.10 (CET)
- net PC_EN: now also U28.10 (CET), U30.10 (CET)
- net at U29.11 (Q3): now also U23.11 (B7)
- net at U29.12 (Q2): now also U23.12 (B6)
- net at U29.13 (Q1): now also U23.13 (B5)
- net at U29.14 (Q0): now also U23.14 (B4)
- net at U29.15 (TC): now also U30.7 (CEP)
- net VCC: now reaches U29.16 (VCC)
- net VCC: now also U28.16 (VCC), U28.7 (CEP), U30.16 (VCC), U23.20 (VCC), U23.20 (VCC)
- net CLK: now reaches U29.2 (CP)
- net CLK: now also U28.2 (CP), U30.2 (CP)
- net at U29.7 (CEP): now also U28.15 (TC)
- net GND: now reaches U29.8 (GND)
- net GND: now also U28.8 (GND), U30.8 (GND), R2.2, R2.2, R2.2, R2.2, R2.2, R2.2, R2.2, R2.2, R2.2, R2.2, R2.2, U23.1 (A->B), U23.1 (A->B), U23.10 (GND), U23.10 (GND)
- net PC_IN: now reaches U29.9 (~{PE})
- net PC_IN: now also U28.9 (~{PE}), U30.9 (~{PE})
- net at U30.11 (Q3): now also U33.1
- net at U30.12 (Q2): now also U23.16 (B2)
- net at U30.13 (Q1): now also U23.17 (B1)
- net at U30.14 (Q0): now also U23.18 (B0)
- net at U28.11 (Q3): now also U23.15 (B3)
- net at U28.12 (Q2): now also U23.16 (B2)
- net at U28.13 (Q1): now also U23.17 (B1)
- net at U28.14 (Q0): now also U23.18 (B0)
- new net: D2.1 (K), R2.1 (x11)
- new net PC_OUT: U23.19 (CE), U23.19 (CE)
- no-connect marks 1 -> 12
Other:
- moved on the sheet: U28, U29, U30
