File: schematics/Clock.kicad_sch (KiCad schematic)
At the start: 0 parts

Commit message: clock
Parts:
- added D54, D55: LED, symbol Device:LED
- added R54, R55, R56, R57, R58, R59, R60, R61: 1k, symbol Device:R
- added RV1: 100k, symbol Device:R_Potentiometer
- added SW1, SW2, SW3, SW4, SW5: SW_Push, symbol Switch:SW_Push
- added U24: ATmega328P-P, Package_DIP:DIP-28_W7.62mm, symbol MCU_Microchip_ATmega:ATmega328P-P
- added U25, U26, U27: 74LS595, symbol 74xx:74LS595
Connections:
- new net: D54.1 (K), R60.2
- new net: D55.1 (K), R61.2
- new net: R59.1, SW5.1, U24.1 (~{RESET}/PC6)
- new net: R54.1, SW1.1, U24.14 (PB0)
- new net: D54.2 (A), U24.5 (PD3), U25.14 (SER), U27.14 (SER)
- new net: RV1.2, U24.24 (PC1)
- new net: R58.1, SW4.1, U24.10 (XTAL2/PB7)
- new net: R56.1, SW2.1, U24.15 (PB1)
- new net: R57.1, SW3.1, U24.9 (XTAL1/PB6)
- new net: U24.12 (PD6), U25.12 (RCLK), U26.12 (RCLK), U27.10 (~{SRCLR})
- new net: U24.6 (PD4), U25.11 (SRCLK), U26.11 (SRCLK), U27.11 (SRCLK)
- new net: U24.4 (PD2), U27.12 (RCLK)
- new net: U24.13 (PD7), U25.13 (~{OE}), U26.13 (~{OE}), U27.13 (~{OE})
- new net: U24.11 (PD5), U25.10 (~{SRCLR}), U26.10 (~{SRCLR})
- new net: U25.9 (QH'), U26.14 (SER)
- new net BUS_0: U27.15 (QA)
- new net BUS_1: U27.1 (QB)
- new net BUS_2: U27.2 (QC)
- new net BUS_3: U27.3 (QD)
- new net BUS_4: U27.4 (QE)
- new net BUS_5: U27.5 (QF)
- new net BUS_6: U27.6 (QG)
- new net BUS_7: U27.7 (QH)
- new net GND: R54.2, R56.2, R57.2, R58.2, R60.1, R61.1, RV1.1, SW5.2, U24.22 (GND), U24.8 (GND), U25.8 (GND), U26.8 (GND), U27.8 (GND)
- new net HLT: D55.2 (A), U24.2 (PD0)
- new net MBUS_0: U25.15 (QA)
- new net MBUS_1: U25.1 (QB)
- new net MBUS_10: U26.2 (QC)
- new net MBUS_2: U25.2 (QC)
- new net MBUS_3: U25.3 (QD)
- new net MBUS_4: U25.4 (QE)
- new net MBUS_5: U25.5 (QF)
- new net MBUS_6: U25.6 (QG)
- new net MBUS_7: U25.7 (QH)
- new net MBUS_8: U26.15 (QA)
- new net MBUS_9: U26.1 (QB)
- new net OLED_SCL: U24.28 (PC5)
- new net OLED_SDA: U24.27 (PC4)
- new net RAM_OE: U24.26 (PC3)
- new net RAM_WE: U24.25 (PC2)
- new net SD_CS: U24.16 (PB2)
- new net SD_MISO: U24.18 (PB4)
- new net SD_MOSI: U24.17 (PB3)
- new net SD_SCK: U24.19 (PB5)
- new net VCC: R59.2, RV1.3, SW1.2, SW2.2, SW3.2, SW4.2, U24.20 (AVCC), U24.7 (VCC), U25.16 (VCC), U26.16 (VCC), U27.16 (VCC)
- no-connect marks 0 -> 8

Commit message: E
Parts:
- removed R58: 1k, symbol Device:R
- removed SW4: SW_Push, symbol Switch:SW_Push
- added C1, C2: 22pF, symbol Device:C
- added D67, D68: LED, symbol Device:LED
- added R73: 1k, symbol Device:R
- added Y1: Crystal, symbol Device:Crystal
Connections:
- net RAM_OE is gone; now on an unnamed net: U24.26 (PC3)
- net GND: now also R55.1, C1.2, C2.2, R73.1
- net HLT: now also U24.3 (PD1); no longer U24.2 (PD0)
- net at R61.2: now also D68.1 (K); no longer D55.1 (K)
- net at R55.2: now also D55.1 (K)
- net at U24.10 (XTAL2/PB7): now also C2.1, Y1.1
- net at R57.1, SW3.1: no longer U24.9 (XTAL1/PB6)
- net CLK: now reaches U24.23 (PC0)
- net CLK: now also D67.2 (A)
- net RAM_WE renamed ~{RAM_WE}
- new net: C1.1, U24.9 (XTAL1/PB6), Y1.2
- new net: D67.1 (K), R73.2
- new net ~{CLK}: D68.2 (A), U24.2 (PD0)
Other:
- moved on the sheet: R54
