File: schematics/ALU.kicad_sch (KiCad schematic)
At the start: 44 parts, among them U10 74LS83, U11 74LS377, U12 74LS377, U13 74LS245, U14 74LS245, U15 74LS08, U16 74LS02, U17 74LS86, U18 74LS86, U7 74LS00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

Commit message: schematics
Other:
- moved on the sheet: U11
Changed lines of the file:
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@@
     (stroke (width 0) (type default))
   )
-  (wire (pts (xy 107.95 199.39) (xy 107.95 196.85))
+  (wire (pts (xy 107.95 201.93) (xy 107.95 196.85))
     (stroke (width 0) (type default))
   )
@@
     (stroke (width 0) (type default))
   )
-  (wire (pts (xy 118.11 224.79) (xy 118.11 279.4))
+  (wire (pts (xy 118.11 227.33) (xy 118.11 279.4))
     (stroke (width 0) (type default))
   )
@@
     (stroke (width 0) (type default))
   )
-  (wire (pts (xy 123.19 224.79) (xy 123.19 248.92))
+  (wire (pts (xy 123.19 227.33) (xy 123.19 248.92))
     (stroke (width 0) (type default))
   )
@@
     (stroke (width 0) (type default))
   )
-  (wire (pts (xy 139.7 212.09) (xy 139.7 204.47))
+  (wire (pts (xy 139.7 214.63) (xy 139.7 207.01))
     (stroke (width 0) (type default))
   )
@@
     (stroke (width 0) (type default))
   )
-  (wire (pts (xy 130.81 138.43) (xy 130.81 199.39))
+  (wire (pts (xy 130.81 138.43) (xy 130.81 201.93))
     (stroke (width 0) (type default))
   )
@@
     (stroke (width 0) (type default))
   )
-  (wire (pts (xy 120.65 148.59) (xy 120.65 199.39))
+  (wire (pts (xy 120.65 148.59) (xy 120.65 201.93))
     (stroke (width 0) (type default))
   )
@@
     (stroke (width 0) (type default))
   )
-  (wire (pts (xy 115.57 224.79) (xy 115.57 275.59))
+  (wire (pts (xy 115.57 227.33) (xy 115.57 275.59))
     (stroke (width 0) (type default))
   )
@@
     (stroke (width 0) (type default))
   )
-  (wire (pts (xy 120.65 224.79) (xy 120.65 283.21))
+  (wire (pts (xy 120.65 227.33) (xy 120.65 283.21))
     (stroke (width 0) (type default))
   )
@@
     (stroke (width 0) (type default))
   )
-  (wire (pts (xy 128.27 199.39) (xy 128.27 140.97))
+  (wire (pts (xy 128.27 201.93) (xy 128.27 140.97))
     (stroke (width 0) (type default))
   )
@@
     (stroke (width 0) (type default))
   )
-  (wire (pts (xy 115.57 153.67) (xy 115.57 199.39))
+  (wire (pts (xy 115.57 153.67) (xy 115.57 201.93))
     (stroke (width 0) (type default))
   )
@@
     (stroke (width 0) (type default))
   )
+  (wire (pts (xy 105.41 201.93) (xy 105.41 199.39))
+    (stroke (width 0) (type default))
+  )
   (wire (pts (xy 199.39 382.27) (xy 172.72 382.27))
     (stroke (width 0) (type default))
@@
     (stroke (width 0) (type default))
   )
-  (wire (pts (xy 138.43 212.09) (xy 139.7 212.09))
+  (wire (pts (xy 138.43 214.63) (xy 139.7 214.63))
     (stroke (width 0) (type default))
   )
@@
     (stroke (width 0) (type default))
   )
-  (wire (pts (xy 125.73 143.51) (xy 125.73 199.39))
+  (wire (pts (xy 125.73 143.51) (xy 125.73 201.93))
     (stroke (width 0) (type default))
   )
@@
     (stroke (width 0) (type default))
   )
-  (wire (pts (xy 123.19 199.39) (xy 123.19 146.05))
+  (wire (pts (xy 123.19 201.93) (xy 123.19 146.05))
     (stroke (width 0) (type default))
   )
@@
     (stroke (width 0) (type default))
   )
-  (wire (pts (xy 125.73 224.79) (xy 125.73 251.46))
+  (wire (pts (xy 125.73 227.33) (xy 125.73 251.46))
     (stroke (width 0) (type default))
   )
@@
     (stroke (width 0) (type default))
   )
-  (wire (pts (xy 93.98 212.09) (xy 97.79 212.09))
+  (wire (pts (xy 93.98 214.63) (xy 97.79 214.63))
     (stroke (width 0) (type default))
   )
@@
     (stroke (width 0) (type default))
   )
-  (wire (pts (xy 128.27 224.79) (xy 128.27 254))
+  (wire (pts (xy 128.27 227.33) (xy 128.27 254))
     (stroke (width 0) (type default))
   )
@@
     (stroke (width 0) (type default))
   )
-  (wire (pts (xy 113.03 224.79) (xy 113.03 271.78))
+  (wire (pts (xy 113.03 227.33) (xy 113.03 271.78))
     (stroke (width 0) (type default))
   )
@@
     (stroke (width 0) (type default))
   )
-  (wire (pts (xy 113.03 199.39) (xy 113.03 156.21))
+  (wire (pts (xy 113.03 201.93) (xy 113.03 156.21))
     (stroke (width 0) (type default))
   )
@@
     (stroke (width 0) (type default))
   )
-  (wire (pts (xy 93.98 214.63) (xy 93.98 212.09))
+  (wire (pts (xy 93.98 217.17) (xy 93.98 214.63))
     (stroke (width 0) (type default))
   )
@@
     (stroke (width 0) (type default))
   )
-  (wire (pts (xy 118.11 199.39) (xy 118.11 151.13))
+  (wire (pts (xy 118.11 201.93) (xy 118.11 151.13))
     (stroke (width 0) (type default))
   )
@@
     (stroke (width 0) (type default))
   )
-  (wire (pts (xy 130.81 224.79) (xy 130.81 256.54))
+  (wire (pts (xy 130.81 227.33) (xy 130.81 256.54))
     (stroke (width 0) (type default))
   )
@@
     )
   )
-  (symbol (lib_id "power:VCC") (at 139.7 204.47 0) (unit 1)
+  (symbol (lib_id "power:VCC") (at 139.7 207.01 0) (unit 1)
     (in_bom yes) (on_board yes) (dnp no) (fields_autoplaced)
-    (property "Reference" "#PWR016" (at 139.7 208.28 0)
+    (property "Reference" "#PWR016" (at 139.7 210.82 0)
       (effects (font (size 1.27 1.27)) hide)
     )
-    (property "Value" "VCC" (at 139.7 200.66 0)
+    (property "Value" "VCC" (at 139.7 203.2 0)
       (effects (font (size 1.27 1.27)))
     )
-    (property "Footprint" "" (at 139.7 204.47 0)
+    (property "Footprint" "" (at 139.7 207.01 0)
       (effects (font (size 1.27 1.27)) hide)
     )
-    (property "Datasheet" "" (at 139.7 204.47 0)
+    (property "Datasheet" "" (at 139.7 207.01 0)
       (effects (font (size 1.27 1.27)) hide)
     )
@@
     )
   )
-  (symbol (lib_id "74xx:74LS377") (at 118.11 212.09 270) (unit 1)
+  (symbol (lib_id "74xx:74LS377") (at 118.11 214.63 270) (unit 1)
     (in_bom yes) (on_board yes) (dnp no) (fields_autoplaced)
-    (property "Reference" "U11" (at 138.43 206.4003 90)
+    (property "Reference" "U11" (at 138.43 208.9403 90)
       (effects (font (size 1.27 1.27)))
     )
-    (property "Value" "74LS377" (at 138.43 208.9403 90)
+    (property "Value" "74LS377" (at 138.43 211.4803 90)
       (effects (font (size 1.27 1.27)))
     )
-    (property "Footprint" "" (at 118.11 212.09 0)
+    (property "Footprint" "" (at 118.11 214.63 0)
       (effects (font (size 1.27 1.27)) hide)
     )
-    (property "Datasheet" "http://www.ti.com/lit/gpn/sn74LS377" (at 118.11 212.09 0)
+    (property "Datasheet" "http://www.ti.com/lit/gpn/sn74LS377" (at 118.11 214.63 0)
       (effects (font (size 1.27 1.27)) hide)
     )
@@
     )
   )
-  (symbol (lib_id "power:GND") (at 93.98 214.63 0) (unit 1)
+  (symbol (lib_id "power:GND") (at 93.98 217.17 0) (unit 1)
     (in_bom yes) (on_board yes) (dnp no) (fields_autoplaced)
-    (property "Reference" "#PWR015" (at 93.98 220.98 0)
+    (property "Reference" "#PWR015" (at 93.98 223.52 0)
       (effects (font (size 1.27 1.27)) hide)
     )
-    (property "Value" "GND" (at 93.98 219.71 0)
+    (property "Value" "GND" (at 93.98 222.25 0)
       (effects (font (size 1.27 1.27)))
     )
-    (property "Footprint" "" (at 93.98 214.63 0)
+    (property "Footprint" "" (at 93.98 217.17 0)
       (effects (font (size 1.27 1.27)) hide)
     )
-    (property "Datasheet" "" (at 93.98 214.63 0)
+    (property "Datasheet" "" (at 93.98 217.17 0)
       (effects (font (size 1.27 1.27)) hide)
     )

Commit message: control logic finished
Connections:
- net ALU_A_IN renamed ~{ALU_A_IN}
- net ALU_B_IN renamed ~{ALU_B_IN}
Changed lines of the file:
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@@
     (effects (font (size 1.27 1.27)) (justify right))
   )
-  (hierarchical_label "ALU_A_IN" (shape input) (at 105.41 199.39 90) (fields_autoplaced)
+  (hierarchical_label "~{ALU_A_IN}" (shape input) (at 105.41 199.39 90) (fields_autoplaced)
     (effects (font (size 1.27 1.27)) (justify left))
   )
@@
     (effects (font (size 1.27 1.27)) (justify left))
   )
-  (hierarchical_label "ALU_B_IN" (shape input) (at 154.94 201.93 90) (fields_autoplaced)
+  (hierarchical_label "~{ALU_B_IN}" (shape input) (at 154.94 201.93 90) (fields_autoplaced)
     (effects (font (size 1.27 1.27)) (justify left))
   )
