File: schematics/I_Reg.kicad_sch (KiCad schematic)
At the start: 0 parts

Commit message: E
Parts:
- added D1 (x2), D2 (x2), D3 (x2), D4 (x2), D5, D6, D7, D8: LED, symbol Device:LED
- added R1 (x2), R2 (x2), R3 (x2), R4 (x2), R5, R6, R60 (x10), R7, R8: 1k, symbol Device:R
- added U1 (x2): 74LS377, symbol 74xx:74LS377
- added U38: 74LS245, symbol 74xx:74LS245
- added U39: 74LS161, symbol 74xx:74LS161
Connections:
- new net: D4.1 (K), R4.1 (x2)
- new net: D4.2 (A), U1.12 (Q4), U38.6 (A4)
- new net: D1.1 (K), R1.1 (x2)
- new net: D1.2 (A), U1.19 (Q7), U38.9 (A7)
- new net: D5.1 (K), R5.1
- new net: D8.1 (K), R8.1
- new net: D7.1 (K), R7.1
- new net: D7.2 (A), U1.5 (Q1), U38.3 (A1)
- new net: D2.1 (K), R2.1 (x2)
- new net: D6.1 (K), R6.1
- new net: D6.2 (A), U1.6 (Q2), U38.4 (A2)
- new net: D2.2 (A), U1.16 (Q6), U38.8 (A6)
- new net: U1.12 (Q4), U1.13 (D4)
- new net: U1.14 (D5), U1.15 (Q5)
- new net: D3.2 (A), U1.15 (Q5), U38.7 (A5)
- new net: U1.16 (Q6), U1.17 (D6)
- new net: U1.18 (D7), U1.19 (Q7)
- new net: D8.2 (A), U1.2 (Q0), U38.2 (A0)
- new net: U1.2 (Q0), U1.3 (D0)
- new net: U1.4 (D1), U1.5 (Q1)
- new net: U1.6 (Q2), U1.7 (D2)
- new net: U1.8 (D3), U1.9 (Q3)
- new net: D5.2 (A), U1.9 (Q3), U38.5 (A3)
- new net: D3.1 (K), R3.1 (x2)
- new net BUS_0: U1.3 (D0)
- new net BUS_1: U1.4 (D1)
- new net BUS_2: U1.7 (D2)
- new net BUS_3: U1.8 (D3)
- new net BUS_4: U1.13 (D4)
- new net BUS_5: U1.14 (D5)
- new net BUS_6: U1.17 (D6)
- new net BUS_7: U1.18 (D7)
- new net CF: R60.2
- new net CLK: U1.11 (CP), U1.11 (CP), U39.2 (CP)
- new net CL_0: D4.2 (A), U39.14 (Q0)
- new net CL_1: D3.2 (A), U39.13 (Q1)
- new net CL_10: R60.2, U38.12 (B6)
- new net CL_11: R60.2, U38.11 (B7)
- new net CL_12: R60.2
- new net CL_2: D2.2 (A), U39.12 (Q2)
- new net CL_3: D1.2 (A), U39.11 (Q3)
- new net CL_4: R60.2, U38.18 (B0)
- new net CL_5: R60.2, U38.17 (B1)
- new net CL_6: R60.2, U38.16 (B2)
- new net CL_7: R60.2, U38.15 (B3)
- new net CL_8: R60.2, U38.14 (B4)
- new net CL_9: R60.2, U38.13 (B5)
- new net GND: R1.2, R1.2, R2.2, R2.2, R3.2, R3.2, R4.2, R4.2, R5.2, R6.2, R60.1, R60.1, R60.1, R60.1, R60.1, R60.1, R60.1, R60.1, R7.2, R8.2, U1.10 (GND), U1.10 (GND), U38.10 (GND), U39.8 (GND)
- new net IR1_IN: U1.1 (~{E})
- new net IR2_IN: U1.1 (~{E})
- new net VCC: R60.1, R60.1, U1.20 (VCC), U1.20 (VCC), U38.1 (A->B), U38.20 (VCC), U39.10 (CET), U39.16 (VCC), U39.7 (CEP), U39.9 (~{PE})
- new net ~{STPC_RESET}: U39.1 (~{MR})
- no-connect marks 0 -> 5

Commit message: control logic finished
Connections:
- net ~{FETCH}: now reaches U38.19 (CE)
- net IR1_IN renamed ~{IR1_IN}
- net IR2_IN renamed ~{IR2_IN}
Changed lines of the file:
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@@
     (effects (font (size 1.27 1.27)) (justify left))
+  )
+  (hierarchical_label "~{FETCH}" (shape input) (at 158.75 83.82 180) (fields_autoplaced)
+    (effects (font (size 1.27 1.27)) (justify right))
   )
   (hierarchical_label "CF" (shape input) (at 184.15 81.28 180) (fields_autoplaced)
@@
     (effects (font (size 1.27 1.27)) (justify right))
   )
-  (hierarchical_label "IR1_IN" (shape input) (at 48.26 83.82 180) (fields_autoplaced)
+  (hierarchical_label "~{IR1_IN}" (shape input) (at 48.26 83.82 180) (fields_autoplaced)
     (effects (font (size 1.27 1.27)) (justify right))
   )
@@
     (effects (font (size 1.27 1.27)) (justify right))
   )
-  (hierarchical_label "IR2_IN" (shape input) (at 83.82 83.82 180) (fields_autoplaced)
+  (hierarchical_label "~{IR2_IN}" (shape input) (at 83.82 83.82 180) (fields_autoplaced)
     (effects (font (size 1.27 1.27)) (justify right))
   )
