File: schematics/schematics.kicad_sch (KiCad schematic)
At the start: 12 parts, among them SW1 SW_Push, U1 LM555xN, U2 LM555xN

Commit message: schematicsscsc
Parts:
- removed C1: 1uF, symbol Device:C_Polarized
- removed C2, C3: 0.01uF, symbol Device:C
- removed C4: 0.1uF, symbol Device:C_Polarized
- removed R1, R2, R4: 1k, symbol Device:R
- removed R3: 1M, symbol Device:R
- removed RV1: 100k, symbol Device:R_Potentiometer
- removed SW1: SW_Push, symbol Switch:SW_Push
- removed U1, U2: LM555xN, Package_DIP:DIP-8_W7.62mm, symbol Timer:LM555xN
Connections:
- no-connect marks 1 -> 0
Other:
- added sheet A Register (A_Reg.kicad_sch)
- added sheet ALU (ALU.kicad_sch)
- added sheet B Register (B_Reg.kicad_sch)
- added sheet C Register (C_Reg.kicad_sch)

Commit message: schematics
Other:
- added sheet Clock (Clock.kicad_sch)
- added sheet F Register (F_Register.kicad_sch)
- added sheet M Register (M Register.kicad_sch)
Changed lines of the file:
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@@
+    )
+  )
+  (sheet (at 143.51 96.52) (size 25.4 50.8) (fields_autoplaced)
+    (stroke (width 0.1524) (type solid))
+    (fill (color 0 0 0 0.0000))
+    (property "Sheetname" "M Register" (at 143.51 95.8084 0)
+      (effects (font (size 1.27 1.27)) (justify left bottom))
+    )
+    (property "Sheetfile" "M Register.kicad_sch" (at 143.51 147.9046 0)
+      (effects (font (size 1.27 1.27)) (justify left top))
+    )
+    (pin "BUS_4" input (at 168.91 109.22 0)
+      (effects (font (size 1.27 1.27)) (justify right))
+    )
+    (pin "BUS_3" input (at 168.91 106.68 0)
+      (effects (font (size 1.27 1.27)) (justify right))
+    )
+    (pin "BUS_5" input (at 168.91 111.76 0)
+      (effects (font (size 1.27 1.27)) (justify right))
+    )
+    (pin "BUS_7" input (at 168.91 116.84 0)
+      (effects (font (size 1.27 1.27)) (justify right))
+    )
+    (pin "BUS_6" input (at 168.91 114.3 0)
+      (effects (font (size 1.27 1.27)) (justify right))
+    )
+    (pin "CLK" input (at 143.51 113.03 180)
+      (effects (font (size 1.27 1.27)) (justify left))
+    )
+    (pin "ML_IN" input (at 143.51 101.6 180)
+      (effects (font (size 1.27 1.27)) (justify left))
+    )
+    (pin "MH_IN" input (at 143.51 99.06 180)
+      (effects (font (size 1.27 1.27)) (justify left))
+    )
+    (pin "MBUS_10" input (at 143.51 142.24 180)
+      (effects (font (size 1.27 1.27)) (justify left))
+    )
+    (pin "MBUS_9" input (at 143.51 139.7 180)
+      (effects (font (size 1.27 1.27)) (justify left))
+    )
+    (pin "MBUS_7" input (at 143.51 134.62 180)
+      (effects (font (size 1.27 1.27)) (justify left))
+    )
+    (pin "MBUS_6" input (at 143.51 132.08 180)
+      (effects (font (size 1.27 1.27)) (justify left))
+    )
+    (pin "MBUS_8" input (at 143.51 137.16 180)
+      (effects (font (size 1.27 1.27)) (justify left))
+    )
+    (pin "MBUS_0" input (at 143.51 116.84 180)
+      (effects (font (size 1.27 1.27)) (justify left))
+    )
+    (pin "MBUS_3" input (at 143.51 124.46 180)
+      (effects (font (size 1.27 1.27)) (justify left))
+    )
+    (pin "MBUS_5" input (at 143.51 129.54 180)
+      (effects (font (size 1.27 1.27)) (justify left))
+    )
+    (pin "MBUS_1" input (at 143.51 119.38 180)
+      (effects (font (size 1.27 1.27)) (justify left))
+    )
+    (pin "MBUS_2" input (at 143.51 121.92 180)
+      (effects (font (size 1.27 1.27)) (justify left))
+    )
+    (pin "MBUS_4" input (at 143.51 127 180)
+      (effects (font (size 1.27 1.27)) (justify left))
+    )
+    (pin "BUS_1" input (at 168.91 101.6 0)
+      (effects (font (size 1.27 1.27)) (justify right))
+    )
+    (pin "BUS_0" input (at 168.91 99.06 0)
+      (effects (font (size 1.27 1.27)) (justify right))
+    )
+    (pin "BUS_2" input (at 168.91 104.14 0)
+      (effects (font (size 1.27 1.27)) (justify right))
+    )
+    (pin "ML_OUT" input (at 143.51 106.68 180)
+      (effects (font (size 1.27 1.27)) (justify left))
+    )
+    (pin "MH_OUT" input (at 143.51 109.22 180)
+      (effects (font (size 1.27 1.27)) (justify left))
+    )
+    (instances
+      (project "schematics"
+        (path "/9826b01a-7fe5-458a-9e88-dd6568b3458a" (page "7"))
+      )
     )
   )
@@
     )
   )
+  (sheet (at 149.86 59.69) (size 12.7 15.24) (fields_autoplaced)
+    (stroke (width 0.1524) (type solid))
+    (fill (color 0 0 0 0.0000))
+    (property "Sheetname" "Clock" (at 149.86 58.9784 0)
+      (effects (font (size 1.27 1.27)) (justify left bottom))
+    )
+    (property "Sheetfile" "Clock.kicad_sch" (at 149.86 75.5146 0)
+      (effects (font (size 1.27 1.27)) (justify left top))
+    )
+    (instances
+      (project "schematics"
+        (path "/9826b01a-7fe5-458a-9e88-dd6568b3458a" (page "8"))
+      )
+    )
+  )
   (sheet (at 203.2 63.5) (size 25.4 25.4) (fields_autoplaced)
     (stroke (width 0.1524) (type solid))
@@
       )
     )
+  )
+  (sheet (at 241.3 63.5) (size 16.51 15.24) (fields_autoplaced)
+    (stroke (width 0.1524) (type solid))
+    (fill (color 0 0 0 0.0000))
+    (property "Sheetname" "F Register" (at 241.3 62.7884 0)
+      (effects (font (size 1.27 1.27)) (justify left bottom))
+    )
+    (property "Sheetfile" "F_Register.kicad_sch" (at 241.3 79.3246 0)
+      (effects (font (size 1.27 1.27)) (justify left top))
+    )
+    (pin "CF" input (at 257.81 66.04 0)
+      (effects (font (size 1.27 1.27)) (justify right))
+    )
+    (pin "ZF" input (at 257.81 68.58 0)
+      (effects (font (size 1.27 1.27)) (justify right))
+    )
+    (pin "ZF_IN" input (at 241.3 68.58 180)
+      (effects (font (size 1.27 1.27)) (justify left))
+    )
+    (pin "CF_IN" input (at 241.3 66.04 180)
+      (effects (font (size 1.27 1.27)) (justify left))
+    )
+    (pin "CLK" input (at 241.3 71.12 180)
+      (effects (font (size 1.27 1.27)) (justify left))
+    )
+    (pin "~{F_IN}" input (at 241.3 74.93 180)
+      (effects (font (size 1.27 1.27)) (justify left))
+    )
+    (instances
+      (project "schematics"
+        (path "/9826b01a-7fe5-458a-9e88-dd6568b3458a" (page "6"))
+      )
+    )

Commit message: clock
Other:
- added sheet Program Counter (PC.kicad_sch)
Changed lines of the file:
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@@
+    )
+  )
+  (sheet (at 85.09 38.1) (size 12.7 3.81) (fields_autoplaced)
+    (stroke (width 0.1524) (type solid))
+    (fill (color 0 0 0 0.0000))
+    (property "Sheetname" "Program Counter" (at 85.09 37.3884 0)
+      (effects (font (size 1.27 1.27)) (justify left bottom))
+    )
+    (property "Sheetfile" "PC.kicad_sch" (at 85.09 42.4946 0)
+      (effects (font (size 1.27 1.27)) (justify left top))
+    )
+    (instances
+      (project "schematics"
+        (path "/9826b01a-7fe5-458a-9e88-dd6568b3458a" (page "9"))
+      )
     )
   )

Commit message: schematics
Other:
- added sheet I Register (I_Reg.kicad_sch)
- sheet F Register ports: added ~{CLK}; removed CLK
- sheet M Register ports: added M_OUT; removed MH_OUT, ML_OUT
- sheet Program Counter ports: added CLK, MBUS_0, MBUS_1, MBUS_10, MBUS_2, MBUS_3, MBUS_4, MBUS_5, MBUS_6, MBUS_7, MBUS_8, MBUS_9, PC_EN, PC_IN, PC_OUT, PC_RST; removed none

Commit message: E
Connections:
- no-connect marks 0 -> 1
Other:
- sheet I Register renamed I Register + Control
- added sheet RAM (RAM.kicad_sch)
- sheet Clock ports: added BUS_0, BUS_1, BUS_2, BUS_3, BUS_4, BUS_5, BUS_6, BUS_7, CLK, HLT, MBUS_0, MBUS_1, MBUS_10, MBUS_2, MBUS_3, MBUS_4, MBUS_5, MBUS_6, MBUS_7, MBUS_8, MBUS_9, ~{CLK}, ~{RAM_WE}; removed none
- sheet I Register + Control ports: added BUS_0, BUS_1, BUS_2, BUS_3, BUS_4, BUS_5, BUS_6, BUS_7, CF, CLK, CL_0, CL_1, CL_10, CL_11, CL_12, CL_13, CL_2, CL_3, CL_4, CL_5, CL_6, CL_7, CL_8, CL_9, IR1_IN, IR2_IN, ZF, ~{STPC_RESET}; removed none

Commit message: control logic finished
Connections:
- no-connect marks 1 -> 0
Other:
- added sheet Control ROM (Con_ROM.kicad_sch)
- sheet ALU ports: added ~{ALU_A_IN}, ~{ALU_B_IN}; removed ALU_A_IN, ALU_B_IN
- sheet F Register ports: added F_OUT; removed none
- sheet I Register + Control ports: added ~{FETCH}, ~{IR1_IN}, ~{IR2_IN}; removed IR1_IN, IR2_IN
- sheet M Register ports: added ~{MH_IN}, ~{ML_IN}; removed MH_IN, ML_IN
- sheet RAM ports: added ~{RAM_CE}; removed ~{RAM_OE}

Commit message: alot of progress
Other:
- added sheet Output (Out.kicad_sch)
Changed lines of the file:
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@@
     (stroke (width 0) (type default))
+  )
+  (sheet (at 300.99 152.4) (size 25.4 26.67) (fields_autoplaced)
+    (stroke (width 0.1524) (type solid))
+    (fill (color 0 0 0 0.0000))
+    (property "Sheetname" "Output" (at 300.99 151.6884 0)
+      (effects (font (size 1.27 1.27)) (justify left bottom))
+    )
+    (property "Sheetfile" "Out.kicad_sch" (at 300.99 179.6546 0)
+      (effects (font (size 1.27 1.27)) (justify left top))
+    )
+    (instances
+      (project "schematics"
+        (path "/9826b01a-7fe5-458a-9e88-dd6568b3458a" (page "13"))
+      )
+    )
   )
   (sheet (at 241.3 245.11) (size 25.4 38.1) (fields_autoplaced)
